File: kicad/zener/zener_power.kicad_sch (KiCad schematic)
At the start: 11 parts

Commit message: NC nets
Parts:
- gave numbers to parts that had none: 11
Connections:
- no-connect marks 0 -> 8
Changed lines of the file:
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@@
   (junction (at 241.3 87.63) (diameter 1.016) (color 0 0 0 0))
   (junction (at 252.73 100.33) (diameter 1.016) (color 0 0 0 0))
+  (no_connect (at 53.34 71.12))
+  (no_connect (at 74.93 173.99))
+  (no_connect (at 78.74 73.66))
+  (no_connect (at 78.74 76.2))
+  (no_connect (at 78.74 78.74))
+  (no_connect (at 78.74 81.28))
+  (no_connect (at 78.74 83.82))
+  (no_connect (at 224.79 129.54))
   (wire (pts (xy 27.94 154.94) (xy 27.94 162.56))
     (stroke (width 0) (type solid) (color 0 0 0 0))
@@
   (symbol (lib_id "SamacSys_Parts:RT0603FRE07270RL") (at 38.1 140.97 270) (unit 1)
     (in_bom yes) (on_board yes)
-    (property "Reference" "R?" (id 0) (at 40.2337 148.7106 90)
+    (property "Reference" "R3" (id 0) (at 40.2337 148.7106 90)
       (effects (font (size 1.27 1.27)) (justify left))
     )
@@
   (symbol (lib_id "SamacSys_Parts:PAT0805E25R0BST1") (at 196.85 87.63 0) (unit 1)
     (in_bom yes) (on_board yes)
-    (property "Reference" "R?" (id 0) (at 205.74 82.0482 0))
+    (property "Reference" "R1" (id 0) (at 205.74 82.0482 0))
     (property "Value" "PAT0805E25R0BST1" (id 1) (at 205.74 84.3469 0))
     (property "Footprint" "RESC2013X46N" (id 2) (at 210.82 86.36 0)
@@
   (symbol (lib_id "SamacSys_Parts:ERA-6VEB1001V") (at 222.25 87.63 0) (unit 1)
     (in_bom yes) (on_board yes)
-    (property "Reference" "R?" (id 0) (at 231.14 82.0482 0))
+    (property "Reference" "R2" (id 0) (at 231.14 82.0482 0))
     (property "Value" "ERA-6VEB1001V" (id 1) (at 231.14 84.3469 0))
     (property "Footprint" "RESC2012X65N" (id 2) (at 236.22 86.36 0)
@@
   (symbol (lib_id "SamacSys_Parts:GRM21BR60J107ME15L") (at 96.52 177.8 0) (unit 1)
     (in_bom yes) (on_board yes)
-    (property "Reference" "C?" (id 0) (at 102.87 171.1006 0))
+    (property "Reference" "C4" (id 0) (at 102.87 171.1006 0))
     (property "Value" "GRM21BR60J107ME15L" (id 1) (at 102.87 173.3993 0))
     (property "Footprint" "CAPC2012X145N" (id 2) (at 105.41 176.53 0)
@@
   (symbol (lib_id "SamacSys_Parts:GRM21BR60J107ME15L") (at 138.43 177.8 0) (unit 1)
     (in_bom yes) (on_board yes)
-    (property "Reference" "C?" (id 0) (at 144.78 171.1006 0))
+    (property "Reference" "C3" (id 0) (at 144.78 171.1006 0))
     (property "Value" "GRM21BR60J107ME15L" (id 1) (at 144.78 173.3993 0))
     (property "Footprint" "CAPC2012X145N" (id 2) (at 147.32 176.53 0)
@@
   (symbol (lib_id "SamacSys_Parts:C0805X105K8RAC7210") (at 201.93 134.62 270) (unit 1)
     (in_bom yes) (on_board yes)
-    (property "Reference" "C?" (id 0) (at 205.1813 139.8206 90)
+    (property "Reference" "C2" (id 0) (at 205.1813 139.8206 90)
       (effects (font (size 1.27 1.27)) (justify left))
     )
@@
   (symbol (lib_id "SamacSys_Parts:C0805X105K8RAC7210") (at 252.73 107.95 270) (unit 1)
     (in_bom yes) (on_board yes)
-    (property "Reference" "C?" (id 0) (at 255.9813 113.1506 90)
+    (property "Reference" "C1" (id 0) (at 255.981 113.151 90)
       (effects (font (size 1.27 1.27)) (justify left))
     )
@@
   (symbol (lib_id "SamacSys_Parts:ADR510ARTZ-REEL7") (at 44.45 173.99 0) (unit 1)
     (in_bom yes) (on_board yes)
-    (property "Reference" "IC?" (id 0) (at 59.69 167.2906 0))
+    (property "Reference" "IC1" (id 0) (at 59.69 167.2906 0))
     (property "Value" "ADR510ARTZ-REEL7" (id 1) (at 59.69 169.5893 0))
     (property "Footprint" "SOT95P237X112-3N" (id 2) (at 71.12 171.45 0)
@@
   (symbol (lib_id "SamacSys_Parts:TLV70012QDCKRQ1") (at 224.79 104.14 270) (unit 1)
     (in_bom yes) (on_board yes)
-    (property "Reference" "IC?" (id 0) (at 228.0413 115.6906 90)
+    (property "Reference" "IC3" (id 0) (at 228.0413 115.6906 90)
       (effects (font (size 1.27 1.27)) (justify left))
     )
@@
   (symbol (lib_id "SamacSys_Parts:LM3940IMP-3.3_NOPB") (at 127 167.64 90) (unit 1)
     (in_bom yes) (on_board yes)
-    (property "Reference" "IC?" (id 0) (at 135.3313 151.2506 90)
+    (property "Reference" "IC2" (id 0) (at 135.3313 151.2506 90)
       (effects (font (size 1.27 1.27)) (justify right))
     )
@@
   (symbol (lib_id "SamacSys_Parts:1734035-2") (at 53.34 83.82 0) (mirror x) (unit 1)
     (in_bom yes) (on_board yes)
-    (property "Reference" "J?" (id 0) (at 66.04 64.4206 0))
+    (property "Reference" "J1" (id 0) (at 66.04 64.4206 0))
     (property "Value" "1734035-2" (id 1) (at 66.04 66.7193 0))
     (property "Footprint" "17340352" (id 2) (at 74.93 86.36 0)
@@
     )
     (path "/18906b50-e48f-4c50-9bdf-5e7a9bbab2b9"
-      (reference "C?") (unit 1) (value "C0805X105K8RAC7210") (footprint "CAPC2012X100N")
+      (reference "C1") (unit 1) (value "C0805X105K8RAC7210") (footprint "CAPC2012X100N")
+    )
+    (path "/eb6cedad-79f3-4b91-af95-5176e62a8c41"
+      (reference "C2") (unit 1) (value "C0805X105K8RAC7210") (footprint "CAPC2012X100N")
+    )
+    (path "/cec7d42d-27c3-441a-ba6d-85311a9c1731"
+      (reference "C3") (unit 1) (value "GRM21BR60J107ME15L") (footprint "CAPC2012X145N")
     )
     (path "/2e4ed844-90de-40ad-bd61-158a04b6da8d"
-      (reference "C?") (unit 1) (value "GRM21BR60J107ME15L") (footprint "CAPC2012X145N")
-    )
-    (path "/cec7d42d-27c3-441a-ba6d-85311a9c1731"
-      (reference "C?") (unit 1) (value "GRM21BR60J107ME15L") (footprint "CAPC2012X145N")
-    )
-    (path "/eb6cedad-79f3-4b91-af95-5176e62a8c41"
-      (reference "C?") (unit 1) (value "C0805X105K8RAC7210") (footprint "CAPC2012X100N")
+      (reference "C4") (unit 1) (value "GRM21BR60J107ME15L") (footprint "CAPC2012X145N")
     )
     (path "/7803ef41-aafc-4390-95ea-2015bba29ffc"
-      (reference "IC?") (unit 1) (value "ADR510ARTZ-REEL7") (footprint "SOT95P237X112-3N")
+      (reference "IC1") (unit 1) (value "ADR510ARTZ-REEL7") (footprint "SOT95P237X112-3N")
     )
     (path "/b39a1b14-8cac-49d2-8b36-1ca117b72ea8"
-      (reference "IC?") (unit 1) (value "LM3940IMP-3.3_NOPB") (footprint "SOT230P700X180-4N")
+      (reference "IC2") (unit 1) (value "LM3940IMP-3.3_NOPB") (footprint "SOT230P700X180-4N")
     )
     (path "/e7a928cb-1d04-47f6-88b8-6a5ab8b94d2c"
-      (reference "IC?") (unit 1) (value "TLV70012QDCKRQ1") (footprint "SOT65P210X110-5N")
+      (reference "IC3") (unit 1) (value "TLV70012QDCKRQ1") (footprint "SOT65P210X110-5N")
     )
     (path "/46eb41e3-6e66-44b2-8f42-ef9b5e3b4b85"
-      (reference "J?") (unit 1) (value "1734035-2") (footprint "17340352")
+      (reference "J1") (unit 1) (value "1734035-2") (footprint "17340352")
+    )
+    (path "/32a78393-7086-4977-b63e-df9278c13d74"
+      (reference "R1") (unit 1) (value "PAT0805E25R0BST1") (footprint "RESC2013X46N")
     )
     (path "/20252eff-1faf-4ac6-9f8d-e3845986ffb3"
-      (reference "R?") (unit 1) (value "ERA-6VEB1001V") (footprint "RESC2012X65N")
-    )
-    (path "/32a78393-7086-4977-b63e-df9278c13d74"
-      (reference "R?") (unit 1) (value "PAT0805E25R0BST1") (footprint "RESC2013X46N")
+      (reference "R2") (unit 1) (value "ERA-6VEB1001V") (footprint "RESC2012X65N")
     )
     (path "/8b1b52fb-178d-4b18-bf61-119b7ba2f615"
-      (reference "R?") (unit 1) (value "RT0603FRE07270RL") (footprint "RESC1608X55N")
-    )
-  )
+      (reference "R3") (unit 1) (value "RT0603FRE07270RL") (footprint "RESC1608X55N")
+    )
+  )
